File: pcb/clover_timer/clover_timer.kicad_sch (KiCad schematic)
At the start: 7 parts, among them IC1 PMS150G-S08, J1 CR2032_Plus, J2 CR2032_Minus, SW1 SW_Push, SW2 SW_Push

Commit message: update pcb, add docs
Parts:
- BZ1: footprint Buzzer_Beeper:Buzzer_D14mm_H7mm_P10mm -> clover_timer:Buzzer
Changed lines of the file:
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@@
       (effects (font (size 1.27 1.27)) (justify right))
     )
-    (property "Footprint" "Buzzer_Beeper:Buzzer_D14mm_H7mm_P10mm" (at 152.4 93.345 90)
+    (property "Footprint" "clover_timer:Buzzer" (at 152.4 93.345 90)
       (effects (font (size 1.27 1.27)) hide)
     )

Commit message: update docs
Parts:
- renumbered BT2 to BT1
Other:
- moved on the sheet: BT1, J1, J2
